File: _autosave-Acorn Joystick Adapter.kicad_pcb (KiCad board)
At the start: 2 copper layers, 64.1 x 38.7 mm, 17 parts, among them J1 BBC Micro, J2 Atari #1, J3 Atari #2, Q1 BC337, Q2 BC337, Q3 BC337

Commit message: Added second joystick port to schematic
Connections:
- net A_GND renamed VREF
