File: Acorn Joystick Adapter.sch (KiCad schematic (older format))
At the start: 32 parts, among them J1 Acorn Computer, J2 Atari #1, J3 Atari #2, J4 Analog, Q1 BC337, Q2 BC337, Q3 BC337, Q4 BC337, Q5 BC337, Q6 BC337

Commit message: Smaller DSUB mounting holes
Parts:
- J4: footprint Pin_Headers:Pin_Header_Straight_1x05_Pitch2.54mm -> Pin_Headers:Pin_Header_Straight_1x06_Pitch2.54mm; symbol Conn_01x05 -> Conn_01x06
Connections:
- net B_PB0: now also J4.4 (Pin_4)
- net GNDA: now also J4.6 (Pin_6); no longer J4.5 (Pin_5)
- net VREF: now also J4.5 (Pin_5); no longer J4.4 (Pin_4)
Changed lines of the file:
@@
 	10050 1950 10200 1950
 $Comp
-L Conn_01x05 J4
+L Conn_01x06 J4
 U 1 1 5BB0FAAF
 P 10350 5800
 F 0 "J4" H 10350 6100 50  0000 C CNN
-F 1 "Analog" H 10350 5500 50  0000 C CNN
-F 2 "Pin_Headers:Pin_Header_Straight_1x05_Pitch2.54mm" H 10350 5800 50  0001 C CNN
+F 1 "Analog" H 10350 5400 50  0000 C CNN
+F 2 "Pin_Headers:Pin_Header_Straight_1x06_Pitch2.54mm" H 10350 5800 50  0001 C CNN
 F 3 "" H 10350 5800 50  0001 C CNN
 	1    10350 5800
@@
 Wire Wire Line
 	10050 5800 10150 5800
-Text GLabel 10050 5900 0    60   BiDi ~ 0
+Text GLabel 10050 6000 0    60   BiDi ~ 0
 VREF
 $Comp
 L GNDA #PWR08
 U 1 1 5BB12497
-P 10050 6100
-F 0 "#PWR08" H 10050 5850 50  0001 C CNN
-F 1 "GNDA" H 10050 5950 50  0000 C CNN
-F 2 "" H 10050 6100 50  0001 C CNN
-F 3 "" H 10050 6100 50  0001 C CNN
-	1    10050 6100
+P 10050 6200
+F 0 "#PWR08" H 10050 5950 50  0001 C CNN
+F 1 "GNDA" H 10050 6050 50  0000 C CNN
+F 2 "" H 10050 6200 50  0001 C CNN
+F 3 "" H 10050 6200 50  0001 C CNN
+	1    10050 6200
 	1    0    0    -1
 $EndComp
 Wire Wire Line
+	10050 6000 10150 6000
+Wire Wire Line
+	10150 6100 10050 6100
+Wire Wire Line
+	10050 6100 10050 6200
+Text GLabel 10050 5900 0    60   Input ~ 0
+B_PB0
+Wire Wire Line
 	10050 5900 10150 5900
-Wire Wire Line
-	10150 6000 10050 6000
-Wire Wire Line
-	10050 6000 10050 6100
 $EndSCHEMATC
