File: Acorn Joystick Adapter.kicad_sch (KiCad schematic)
At the start: 32 parts, among them J1 Acorn Computer, J2 Atari #1, J3 Atari #2, J4 Analog, Q1 BC337, Q2 BC337, Q3 BC337, Q4 BC337, Q5 BC337, Q6 BC337

Commit message: Updated project for recent version of KiCAD
Parts:
- J4: footprint Connector_PinHeader_2.54mm:PinHeader_1x06_P2.54mm_Horizontal -> Connector_PinHeader_2.54mm:PinHeader_1x06_P2.54mm_Vertical
Changed lines of the file:
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@@
 			)
 		)
-		(property "Footprint" "Connector_PinHeader_2.54mm:PinHeader_1x06_P2.54mm_Horizontal"
+		(property "Footprint" "Connector_PinHeader_2.54mm:PinHeader_1x06_P2.54mm_Vertical"
 			(at 266.7 147.32 0)
 			(effects
